File: hardware/microcomputer/microcomputer.kicad_sch (KiCad schematic)
At the start: 91 parts, among them SW1 SW_SPST, SW10 SW_SPST, SW11 SW_SPST, SW12 SW_SPST, SW13 SW_SPST, SW14 SW_SPST, SW15 SW_SPST, SW16 SW_SPST, SW17 KEY, SW18 AUTO INCREMENT, SW19 SINGLE STEP, SW2 SW_SPST, SW20 RESET, SW21 STORE ADDR, SW22 STORE BYTE, SW23 STORE WORD, SW24 RUN SLOW/STOP/RUN FAST, SW3 SW_SPST, SW4 SW_SPST, SW5 SW_SPST, SW6 SW_SPST, SW7 SW_SPST, SW8 SW_SPST, SW9 SW_SPST, U1 74HCT595, U2 74HCT595, U3 PCF8574T, U4 PCF8574T, U5 NHD-0420H1Z

Commit message: Update schematic
Parts:
- added J1: Conn_01x03, symbol Connector_Generic:Conn_01x03
Connections:
- net +5V: now also J1.1 (Pin_1)
- net GND: now also J1.3 (Pin_3)
Other:
- note added: "20x2 LCD (parallel)"
- note added: "CU20025SCPB LCD (serial)"
- note removed: "20x2 LCD"
